File: source/Cheap FOCer 2 60mm.kicad_pcb (KiCad board)
At the start: 2 copper layers, 59.1 x 99.9 mm, 193 parts, among them J1 Conn_01x02, J2 Conn_01x07, J3 Conn_01x03, J4 On/Off, J5 UNUSED MCU PINS, J6 Conn_01x03, P1 MOTOR1, P2 MOTOR1, P3 MOTOR1, P4 HALL/Encoder, P5 SWD, Q1 NCEP60T20, Q2 NCEP60T20, Q3 NCEP60T20, Q4 NCEP60T20, Q5 NCEP60T20, Q6 NCEP60T20, U1 AMS1117-3.3, U2 DRV8301, U3 TP2604-SR, U4 TJA1051T/3/1J, U5 STM32F405RGT6, U6 BMI160, X1 8MHz 10ppm (X50328MSB2GI)

Commit message: V1.0
V1.0
Parts:
- removed H7: MountingHole, MountingHole:MountingHole_3.2mm_M3_ISO14580_Pad
- added C68: 4.7nF, 100V, Capacitor_SMD:C_0805_2012Metric, F.Cu at (128.7, 90.7)
- added C69: 330u, 63V, shapes3D:CP_10x20mm_hor_with_model_mirrored_less_silk, F.Cu at (152.4, 77.3)
- added C70: 4.7nF, 100V, Capacitor_SMD:C_0805_2012Metric, F.Cu at (148.7, 91.1)
- added C71: 4.7nF, 100V, Capacitor_SMD:C_0805_2012Metric, F.Cu at (167.9, 90.7)
- added C72: 220n, Capacitor_SMD:C_0603_1608Metric, F.Cu at (157.3, 153.8)
- added C73: 100n, Capacitor_SMD:C_0603_1608Metric, F.Cu at (134.2, 161.8)
- added C74: 100n, Capacitor_SMD:C_0603_1608Metric, F.Cu at (133.8, 160.3)
- added C75: 100n, Capacitor_SMD:C_0603_1608Metric, F.Cu at (132.9, 158.8)
- added D10: D_Schottky, Diode_SMD:D_SOD-323, F.Cu at (145.6, 93.4)
- added D11: D_Schottky, Diode_SMD:D_SOD-323, F.Cu at (164.9, 93.4)
- added D12: D_Schottky, Diode_SMD:D_SOD-323, F.Cu at (157.2, 109.6)
- added D13: D_TVS, Diode_SMD:D_SMB, F.Cu at (130.2, 131.6)
- added D7: D_Schottky, Diode_SMD:D_SOD-323, F.Cu at (117.7, 109.8)
- added D8: D_Schottky, Diode_SMD:D_SOD-323, F.Cu at (125.4, 93.4)
- added D9: D_Schottky, Diode_SMD:D_SOD-323, F.Cu at (138.4, 109.5)
- added Q10: Q_PNP_BCE, Package_TO_SOT_SMD:SOT-23, F.Cu at (148.6, 93.8)
- added Q11: Q_PNP_BCE, Package_TO_SOT_SMD:SOT-23, F.Cu at (167.7, 93.4)
- added Q12: Q_PNP_BCE, Package_TO_SOT_SMD:SOT-23, F.Cu at (154.5, 109.6)
- added Q7: Q_PNP_BCE, Package_TO_SOT_SMD:SOT-23, F.Cu at (115.1, 109.9)
- added Q8: Q_PNP_BCE, Package_TO_SOT_SMD:SOT-23, F.Cu at (128.4, 93.4)
- added Q9: Q_PNP_BCE, Package_TO_SOT_SMD:SOT-23, F.Cu at (135.7, 109.5)
- added R73: 10R, Resistor_SMD:R_0805_2012Metric, F.Cu at (128.7, 88.8)
- added R74: 10R, Resistor_SMD:R_0805_2012Metric, F.Cu at (128.7, 86.9)
- added R75: 4.7R, Resistor_SMD:R_0603_1608Metric, F.Cu at (120.2, 111.9)
- added R76: 4.7R, Resistor_SMD:R_0603_1608Metric, F.Cu at (127.9, 98.8)
- added R77: 4.7R, Resistor_SMD:R_0603_1608Metric, F.Cu at (139.9, 111.6)
- added R78: 4.7R, Resistor_SMD:R_0603_1608Metric, F.Cu at (148.4, 99.9)
- added R79: 4.7R, Resistor_SMD:R_0603_1608Metric, F.Cu at (168.0, 99.1)
- added R80: 4.7R, Resistor_SMD:R_0603_1608Metric, F.Cu at (151.3, 110.6)
- added R81: 10R, Resistor_SMD:R_0805_2012Metric, F.Cu at (148.7, 89.2)
- added R82: 10R, Resistor_SMD:R_0805_2012Metric, F.Cu at (148.7, 87.3)
- added R83: 10R, Resistor_SMD:R_0805_2012Metric, F.Cu at (167.9, 87.0)
- added R84: 10R, Resistor_SMD:R_0805_2012Metric, F.Cu at (167.9, 88.8)
- added R85: 100R, Resistor_SMD:R_0603_1608Metric, F.Cu at (146.8, 159.6)
- added R86: 100R, Resistor_SMD:R_0603_1608Metric, F.Cu at (146.8, 161.1)
- added R87: 100R, Resistor_SMD:R_0603_1608Metric, F.Cu at (146.8, 162.6)
- C13: value 120p -> 150p
- C15, C31: footprint Capacitor_SMD:C_1210_3225Metric -> Capacitor_SMD:C_1210_3225Metric_Pad1.42x2.65mm_HandSolder
- C38, C39: footprint w_capacitors:CP_10x20mm_hor_with_model_brd_edge -> shapes3D:CP_10x20mm_hor_with_model_mirrored_less_silk
- C61, C62, C63, C65: value 1nF -> 2.2nF
- J3: footprint Connector_JST:JST_PH_B3B-PH-K_1x03_P2.00mm_Vertical -> shapes3D:JST_PH_B3B-PH-K_1x03_P2.00mm_Vertical_hybrid
- POS1: moved to F.Cu
- R26, R28, R30: value 1k -> 1.5k
- R41, R42, R43, R47, R48, R49: value 10R -> 4.7R
- R56, R57, R58, R59, R60, R61: value 0.001R -> 0.002R
- R64, R65: value 20k -> 10k
- moved C39 28.1 mm to (134.0, 77.4)
- moved C38 19.6 mm to (115.6, 77.4)
- moved R17 18.9 mm to (152.0, 161.7), turned to 270 degrees
- moved R16 17.2 mm to (150.5, 161.7), turned to 270 degrees
- moved R15 15.7 mm to (149.0, 161.7), turned to 270 degrees
- moved D1 8.35 mm to (154.3, 160.7)
- moved NT1 5.20 mm to (114.7, 102.5)
- moved R56 5.15 mm to (116.7, 101.6)
- moved R57 5.15 mm to (112.8, 101.6)
- moved R58 5.14 mm to (137.0, 101.5)
- moved R59 5.14 mm to (133.2, 101.5)
- moved NT2 5.13 mm to (135.1, 102.4)
- moved NT5 5.13 mm to (135.1, 100.6)
- moved R60 5.12 mm to (152.5, 101.5)
- moved R61 5.12 mm to (156.4, 101.5)
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Connections:
- D1 pad 6: /HALL3 -> /Filters/HALL3_IN
- J2 pad 1: /MISO_RX_SCL_IN -> +5V
- J2 pad 2: /TX_SCL_MOSI_IN -> VCC
- J2 pad 3: /RX_SDA_IN -> GND
- J2 pad 5: GND -> /RX_SDA_IN
- J2 pad 6: VCC -> /TX_SCL_MOSI_IN
- J2 pad 7: +5V -> /MISO_RX_SCL_IN
- P4 pad 2: /HALL3 -> /Filters/HALL3_IN
- R15 pad 1: /HALL3 -> /Filters/HALL3_IN
- U5 pad 37: /Filters/HALL1_IN -> /Filters/HALL1_OUT
- U5 pad 38: /Filters/HALL2_IN -> /Filters/HALL2_OUT
Routing:
- net GND: track 236.2 -> 267.1 mm, vias 383 -> 510
- net /Filters/HALL1_OUT: track 0.00 -> 21.5 mm
- net /Mosfet driver/H1_VS: track 52.7 -> 72.1 mm, vias 19 -> 20
- net /Mosfet driver/H2_VS: track 45.6 -> 64.7 mm, vias 18 -> 20
- net /Filters/HALL3_IN: track 0.00 -> 18.9 mm
- net /Filters/HALL2_OUT: track 0.00 -> 17.8 mm
- net V_SUPPLY: track 143.5 -> 157.5 mm, vias 75 -> 59
- net /HALL3: track 30.9 -> 17.0 mm
- net /Filters/TEMP_IN: track 41.1 -> 54.1 mm
- net VCC: track 358.3 -> 346.3 mm, vias 31 -> 29
- net /Mosfet driver/H3_VS: track 80.5 -> 90.4 mm, vias 19 -> 21
- net Net-(C62-Pad1): track 5.15 -> 14.6 mm
- net /Filters/HALL2_IN: track 28.4 -> 19.1 mm, vias 3 -> 0
- net /Filters/HALL1_IN: track 30.6 -> 21.7 mm, vias 2 -> 0
- net /TX_SCL_MOSI_IN: track 13.0 -> 21.1 mm
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Other:
- rule trace_min: 0.1778 -> 0
