File: source/Cheap FOCer 2 60mm.sch (KiCad schematic (older format))
At the start: 49 parts, among them J1 Conn_01x02, J2 Conn_01x07, J3 Conn_01x03, J6 Conn_01x03, P1 MOTOR1, P2 MOTOR1, P3 MOTOR1, P4 HALL/Encoder

Commit message: V1.0
V1.0
Parts:
- removed H7: MountingHole, MountingHole:MountingHole_3.2mm_M3_ISO14580_Pad, symbol Mechanical:MountingHole_Pad
- J3: footprint Connector_JST:JST_PH_B3B-PH-K_1x03_P2.00mm_Vertical -> shapes3D:JST_PH_B3B-PH-K_1x03_P2.00mm_Vertical_hybrid
Changed lines of the file:
@@
 	1    0    0    -1
-$EndComp
-$Comp
-L Mechanical:MountingHole_Pad H7
-U 1 1 5DC3863B
-P 12300 3600
-F 0 "H7" V 12300 3750 50  0000 L CNN
-F 1 "MountingHole" H 12400 3555 50  0001 L CNN
-F 2 "MountingHole:MountingHole_3.2mm_M3_ISO14580_Pad" H 12300 3600 50  0001 C CNN
-F 3 "~" H 12300 3600 50  0001 C CNN
-	1    12300 3600
-	0    1    1    0
 $EndComp
 Wire Wire Line
@@
 F 3 "~" H 2900 7750 50  0001 C CNN
 	1    2900 7750
-	-1   0    0    1
+	-1   0    0    -1
 $EndComp
 $Comp
@@
 F 0 "J3" H 10368 7325 50  0000 C CNN
 F 1 "Conn_01x03" H 10368 7416 50  0000 C CNN
-F 2 "Connector_JST:JST_PH_B3B-PH-K_1x03_P2.00mm_Vertical" H 10450 7650 50  0001 C CNN
+F 2 "shapes3D:JST_PH_B3B-PH-K_1x03_P2.00mm_Vertical_hybrid" H 10450 7650 50  0001 C CNN
 F 3 "~" H 10450 7650 50  0001 C CNN
 	1    10450 7650
@@
 Wire Wire Line
 	5550 3650 5750 3650
-Connection ~ 12200 3600
 Wire Wire Line
 	3200 6450 4100 6450
