File: source/Power.sch (KiCad schematic (older format))
At the start: 60 parts, among them J4 On/Off, U1 AMS1117-3.3, U2 DRV8301, U3 TP2604-SR

Commit message: V1.0
V1.0
Parts:
- added C72: 220n, Capacitor_SMD:C_0603_1608Metric, symbol BLDC_4-rescue:C-RESCUE-BLDC_4
- added D13: D_TVS, Diode_SMD:D_SMB, symbol Device:D_TVS
- C15, C31: footprint Capacitor_SMD:C_1210_3225Metric -> Capacitor_SMD:C_1210_3225Metric_Pad1.42x2.65mm_HandSolder
- R26, R28, R30: value 1k -> 1.5k
- R64, R65: value 20k -> 10k
Connections:
- net +5V: now also D13.1 (A1)
- net GND: now also C72.1, D13.2 (A2)
- net at J4.1 (A), U2.55 (EN_BUCK): now also C72.2
Changed lines of the file:
@@
 	1    0    0    -1
 $EndComp
-Text GLabel 10900 2700 0    60   Input ~ 0
+Text GLabel 11000 2950 0    60   Input ~ 0
 V_SUPPLY
 Text HLabel 4750 2150 0    60   Output ~ 0
@@
 F 0 "C31" H 6650 4550 50  0000 L CNN
 F 1 "4.7uF, 100V" H 6700 4850 50  0000 L CNN
-F 2 "Capacitor_SMD:C_1210_3225Metric" H 6650 4650 60  0001 C CNN
+F 2 "Capacitor_SMD:C_1210_3225Metric_Pad1.42x2.65mm_HandSolder" H 6650 4650 60  0001 C CNN
 F 3 "" H 6650 4650 60  0001 C CNN
 	1    6650 4650
@@
 	11050 2550 11050 2700
 Wire Wire Line
-	11050 2700 10900 2700
+	11050 2700 11000 2950
 Text GLabel 7950 1400 2    60   Input ~ 0
 V_SUPPLY
@@
 	7650 2250 8400 2250
 Wire Wire Line
-	7050 1250 7250 1250
+	7050 1250 7200 1250
 Wire Wire Line
 	6750 1850 6900 1850
@@
 $EndComp
 Wire Wire Line
-	7650 1250 8050 1250
+	7650 1250 7750 1250
 $Comp
 L BLDC_4-rescue:C-RESCUE-BLDC_4 C?
@@
 F 0 "C15" H 7600 1600 50  0000 L CNN
 F 1 "4.7uF, 100V" H 7300 1800 50  0000 L CNN
-F 2 "Capacitor_SMD:C_1210_3225Metric" H 7800 1700 60  0001 C CNN
+F 2 "Capacitor_SMD:C_1210_3225Metric_Pad1.42x2.65mm_HandSolder" H 7800 1700 60  0001 C CNN
 F 3 "" H 7800 1700 60  0001 C CNN
 	1    7800 1700
@@
 L power:+5V #PWR035
 U 1 1 5DA1095B
-P 10200 2250
-F 0 "#PWR035" H 10200 2340 20  0001 C CNN
-F 1 "+5V" H 10200 2400 30  0000 C CNN
-F 2 "" H 10200 2250 60  0001 C CNN
-F 3 "" H 10200 2250 60  0001 C CNN
-	1    10200 2250
+P 10600 2250
+F 0 "#PWR035" H 10600 2340 20  0001 C CNN
+F 1 "+5V" H 10600 2400 30  0000 C CNN
+F 2 "" H 10600 2250 60  0001 C CNN
+F 3 "" H 10600 2250 60  0001 C CNN
+	1    10600 2250
 	0    1    1    0
 $EndComp
@@
 Connection ~ 10100 2250
 Wire Wire Line
-	10100 2250 10200 2250
+	10100 2250 10400 2250
 Wire Wire Line
 	10100 2700 10100 2750
@@
 P 2250 6100
 F 0 "R64" V 2350 6100 50  0000 C CNN
-F 1 "20k" V 2250 6100 50  0000 C CNN
+F 1 "10k" V 2250 6100 50  0000 C CNN
 F 2 "Resistor_SMD:R_0603_1608Metric" H 2250 6100 60  0001 C CNN
 F 3 "" H 2250 6100 60  0001 C CNN
@@
 P 2350 6950
 F 0 "R65" V 2450 6950 50  0000 C CNN
-F 1 "20k" V 2350 6950 50  0000 C CNN
+F 1 "10k" V 2350 6950 50  0000 C CNN
 F 2 "Resistor_SMD:R_0603_1608Metric" H 2350 6950 60  0001 C CNN
 F 3 "" H 2350 6950 60  0001 C CNN
@@
 P 4800 4050
 F 0 "R26" V 4900 4100 50  0000 C CNN
-F 1 "1k" V 4800 4050 50  0000 C CNN
+F 1 "1.5k" V 4800 4050 50  0000 C CNN
 F 2 "Resistor_SMD:R_0603_1608Metric" H 4800 4050 60  0001 C CNN
 F 3 "" H 4800 4050 60  0001 C CNN
@@
 P 4800 4150
 F 0 "R28" V 4700 4200 50  0000 C CNN
-F 1 "1k" V 4800 4150 50  0000 C CNN
+F 1 "1.5k" V 4800 4150 50  0000 C CNN
 F 2 "Resistor_SMD:R_0603_1608Metric" H 4800 4150 60  0001 C CNN
 F 3 "" H 4800 4150 60  0001 C CNN
@@
 P 1600 6500
 F 0 "R30" V 1550 6700 50  0000 C CNN
-F 1 "1k" V 1600 6500 50  0000 C CNN
+F 1 "1.5k" V 1600 6500 50  0000 C CNN
 F 2 "Resistor_SMD:R_0603_1608Metric" H 1600 6500 60  0001 C CNN
 F 3 "" H 1600 6500 60  0001 C CNN
@@
 Wire Wire Line
 	4850 4250 4850 4500
+$Comp
+L BLDC_4-rescue:C-RESCUE-BLDC_4 C72
+U 1 1 5EF1C5FE
+P 7500 800
+F 0 "C72" V 7550 600 50  0000 L CNN
+F 1 "220n" V 7450 550 50  0000 L CNN
+F 2 "Capacitor_SMD:C_0603_1608Metric" H 7500 800 60  0001 C CNN
+F 3 "" H 7500 800 60  0001 C CNN
+	1    7500 800
+	0    1    1    0
+$EndComp
+Wire Wire Line
+	7300 800  7200 800
+Wire Wire Line
+	7200 800  7200 1250
+Connection ~ 7200 1250
+Wire Wire Line
+	7200 1250 7250 1250
+Wire Wire Line
+	7700 800  7750 800
+Wire Wire Line
+	7750 800  7750 1250
+Connection ~ 7750 1250
+Wire Wire Line
+	7750 1250 8050 1250
+$Comp
+L Device:D_TVS D13
+U 1 1 5F2D96BD
+P 10400 2500
+F 0 "D13" V 10354 2579 50  0000 L CNN
+F 1 "D_TVS" V 10445 2579 50  0000 L CNN
+F 2 "Diode_SMD:D_SMB" H 10400 2500 50  0001 C CNN
+F 3 "~" H 10400 2500 50  0001 C CNN
+	1    10400 2500
+	0    1    1    0
+$EndComp
+Wire Wire Line
+	10400 2250 10400 2350
+Connection ~ 10400 2250
+Wire Wire Line
+	10400 2250 10600 2250
+Wire Wire Line
+	10400 2650 10400 2750
+Wire Wire Line
+	10400 2750 10100 2750
+Connection ~ 10100 2750
 $EndSCHEMATC
