File: source/mosfets.sch (KiCad schematic (older format))
At the start: 50 parts, among them Q1 NCEP60T20, Q2 NCEP60T20, Q3 NCEP60T20, Q4 NCEP60T20, Q5 NCEP60T20, Q6 NCEP60T20

Commit message: V1.0
V1.0
Parts:
- added C68, C70, C71: 4.7nF, 100V, Capacitor_SMD:C_0805_2012Metric, symbol BLDC_4-rescue:C-RESCUE-BLDC_4
- added C69: 330u, 63V, shapes3D:CP_10x20mm_hor_with_model_mirrored_less_silk, symbol Device:CP1
- added D10, D11, D12, D7, D8, D9: D_Schottky, Diode_SMD:D_SOD-323, symbol Device:D_Schottky
- added Q10, Q11, Q12, Q7, Q8, Q9: Q_PNP_BCE, Package_TO_SOT_SMD:SOT-23, symbol Device:Q_PNP_BEC
- added R73, R74, R81, R82, R83, R84: 10R, Resistor_SMD:R_0805_2012Metric, symbol BLDC_4-rescue:R-RESCUE-BLDC_4
- added R75, R76, R77, R78, R79, R80: 4.7R, Resistor_SMD:R_0603_1608Metric, symbol BLDC_4-rescue:R-RESCUE-BLDC_4
- C38, C39: footprint w_capacitors:CP_10x20mm_hor_with_model_brd_edge -> shapes3D:CP_10x20mm_hor_with_model_mirrored_less_silk
- C61, C62, C63, C65: value 1nF -> 2.2nF
- R41, R42, R43, R47, R48, R49: value 10R -> 4.7R
Connections:
- net GH_A: now also R76.2
- net GH_B: now also R78.2
- net GH_C: now also R79.2
- net GL_A: now also R75.2
- net GL_B: now also R77.2
- net GL_C: now also R80.2
- net GND: now also C69.2
- net H1_LOW: now also D7.2 (A), Q7.3 (C)
- net H1_VS: now also C68.1, D8.2 (A), Q8.3 (C)
- net H2_LOW: now also D9.2 (A), Q9.3 (C)
- net H2_VS: now also C70.1, D10.2 (A), Q10.3 (C)
- net H3_LOW: now also D12.2 (A), Q12.3 (C)
- net H3_VS: now also C71.1, D11.2 (A), Q11.3 (C)
- net V_SUPPLY: now also C69.1, R73.1, R74.1, R81.1, R82.1, R83.1, R84.1
- net at C61.1, Q1.1 (G), R41.1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: now also D8.1 (K), Q8.2 (E)
- net at C62.1, Q4.1 (G), R47.1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: now also D7.1 (K), Q7.2 (E)
- net at C65.1, Q5.1 (G), R48.1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: now also D9.1 (K), Q9.2 (E)
- net at C63.1, Q2.1 (G), R42.1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: now also D10.1 (K), Q10.2 (E)
- net at C66.1, Q3.1 (G), R43.1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: now also D11.1 (K), Q11.2 (E)
- net at C67.1, Q6.1 (G), R49.1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: now also D12.1 (K), Q12.2 (E)
- new net: Q8.1 (B), R76.1
- new net: Q7.1 (B), R75.1
- new net: C68.2, R73.2, R74.2
- new net: Q10.1 (B), R78.1
- new net: Q11.1 (B), R79.1
- new net: Q12.1 (B), R80.1
- new net: Q9.1 (B), R77.1
- new net: C70.2, R81.2, R82.2
- new net: C71.2, R83.2, R84.2
Other:
- moved on the sheet: C38, C40, C42, C61, C62, C66, C67, NT1, NT3, NT4, NT6, Q1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
